Commit message: shoe packing add label v5.0 and kitchen setting v3.0

File: bulletarm/pybullet/urdf/object/kitchen_set/lobster_plate/lobster_plate.urdf (robot description, URDF)
Before this commit: robot plate.urdf, 1 links, 0 joints
Links:
- removed link plateLink
- added link lobsterPlateLink, mass 0; collision mesh filename=lobster_plate.obj scale=0.02 0.02 0.02; visual mesh filename=lobster_plate.obj scale=0.02 0.02 0.02
