Commit message: shoe packing add label v5.0 and kitchen setting v1.0

File: bulletarm/pybullet/urdf/object/kitchen_set/plate/plate.urdf (robot description, URDF)
Before this commit: robot plate.urdf, 1 links, 0 joints
Links:
- link plateLink: geometry collision mesh filename=plate.obj scale=1 1.4 1; visual mesh filename=plate.obj scale=1 1.4 1
