Commit message: kitchen set adjustment urdf

File: bulletarm/pybullet/urdf/object/kitchen_set/knife/knife.urdf (robot description, URDF)
Before this commit: robot knife.urdf, 1 links, 0 joints
Links:
- removed link knifeLink
- added link knifeBase, mass .2; collision box size=0.1 0.02 0.03; visual mesh filename=knife.obj scale=0.02 0.02 0.03
- added link knifeGrasp, mass 0
Joints:
- added joint base2left: type fixed, parent knifeBase, child knifeGrasp, origin xyz=-0.03 0 0 rpy=0 0 0

File: bulletarm/pybullet/urdf/object/kitchen_set/lobster_plate/lobster_plate.urdf (robot description, URDF)
Before this commit: robot lobsterPlate.urdf, 1 links, 0 joints
Links:
- removed link lobsterPlateLink
- added link lobsterPlateBase, mass 0; collision mesh filename=lobster_plate.obj scale=0.02 0.02 0.02; visual mesh filename=lobster_plate.obj scale=0.02 0.02 0.02
- added link lobsterPlateLeft, mass 0; visual box size=0.01 0.01 0.01
- added link lobsterPlateRight, mass 0; visual box size=0.01 0.01 0.01
Joints:
- added joint base2left: type fixed, parent lobsterPlateBase, child lobsterPlateLeft, origin xyz=0 -0.12 0 rpy=0 0 0
- added joint base2right: type fixed, parent lobsterPlateBase, child lobsterPlateRight, origin xyz=0 0.12 0 rpy=0 0 0
