Commit message: kitchen setting env update v2.0

File: bulletarm/pybullet/urdf/object/kitchen_set/fork/fork.urdf (robot description, URDF)
Before this commit: robot fork.urdf, 1 links, 0 joints
Links:
- link forkLink: geometry collision mesh filename=fork.obj scale=1 1 1; visual mesh filename=fork.obj scale=1 1 1

File: bulletarm/pybullet/urdf/object/kitchen_set/knife/knife.urdf (robot description, URDF)
Before this commit: robot knife.urdf, 1 links, 0 joints
Links:
- link knifeLink: geometry collision mesh filename=knife.obj scale=0.02 0.02 0.02; visual mesh filename=knife.obj scale=0.02 0.02 0.02

File: bulletarm/pybullet/urdf/object/kitchen_set/plate/plate.urdf (robot description, URDF)
Before this commit: robot plate.urdf, 1 links, 0 joints
Links:
- link plateLink: geometry collision mesh filename=plate.obj scale=1 1 1; visual mesh filename=plate.obj scale=1 1 1

Commit message: kitchen update

File: bulletarm/pybullet/urdf/object/kitchen_set/fork/fork.urdf (robot description, URDF)
Before this commit: robot fork.urdf, 1 links, 0 joints
Links:
- link forkLink: mass .1 -> .2; geometry collision box size=0.08 0.015 0.02; collision mesh filename=fork.obj scale=1 1 1

File: bulletarm/pybullet/urdf/object/kitchen_set/knife/knife.urdf (robot description, URDF)
Before this commit: robot knife.urdf, 2 links, 1 joints
Links:
- link knifeBase: geometry collision box size=0.08 0.02 0.02; collision mesh filename=knife.obj scale=0.02 0.02 0.04
- link knifeGrasp: geometry visual box size=0.01 0.01 0.01
Joints:
- removed joint base2left
- added joint base2grasp: type fixed, parent knifeBase, child knifeGrasp, origin xyz=-0.035 0 0 rpy=0 0 0

File: bulletarm/pybullet/urdf/object/kitchen_set/lobster_plate/lobster_plate.urdf (robot description, URDF)
Before this commit: robot lobsterPlate.urdf, 3 links, 2 joints
Links:
- link lobsterPlateLeft: geometry 
- link lobsterPlateRight: geometry 
Joints:
- joint base2left: origin xyz=0 -0.12 0 rpy=0 0 0 -> xyz=0 -0.12 -0.02 rpy=0 0 0
- joint base2right: origin xyz=0 0.12 0 rpy=0 0 0 -> xyz=0.035 0.12 -0.02 rpy=0 0 0
